File: board-basetation/wifibasestation.sch (EAGLE design)
At the start: 33 parts, among them IC1 1117EMP, IC2 HTU21D, J1 SWD_SHROUD_SMD, X1 ESP-03, X2 SMA-142-0711-821/826

Commit message: pretty much done
Parts:
- removed C11: (no value), rcl:C-EUC0603K
- removed U$3: LMT85, Mine:LMT85
- added C7: 1u, rcl:C-EUC0603
- added IC3: HTU21D, Mine:HTU21D
- C1, C5: value (none) -> 4u7; device rcl:C-EUC0603K -> rcl:C-EUC0603
- C10, C2, C3: value (none) -> 1u; device rcl:C-EUC0603K -> rcl:C-EUC0603
- C4, C8, C9: value (none) -> 100n; device rcl:C-EUC0603K -> rcl:C-EUC0603
- C6: value (none) -> 100n
- IC2: value HTU21D -> STM32F072; device Mine:HTU21D -> dtb:STM32F072
- JP3: value FTDI_BASICPTH -> USB-A-H; device SparkFun-Connectors:FTDI_BASICPTH -> SparkFun-Connectors:USB-A-H
- JP4: value USB-A-H -> FTDI_BASICPTH; device SparkFun-Connectors:USB-A-H -> SparkFun-Connectors:FTDI_BASICPTH
- R1, R2: value (none) -> 10k
- R3: value (none) -> 100k
- R4, R5: value (none) -> 4k7
- RN1: value (none) -> 330
- U$1: value STM32F072 -> LMT85; device dtb:STM32F072 -> Mine:LMT85
- renumbered S2 to S1
Connections:
- net +3V3: now also C2.1, C7.1, C8.1, IC2.VDD(VBAT), IC2.VDD1, IC2.VDDA, IC3.VDD, JP4.4, R4.2; no longer C1.1, C11.1, C6.1, JP3.4, R1.2, U$1.VDD, U$1.VDD(VBAT), U$1.VDD1, U$1.VDDA
- net CH_PD: now also IC2.PF0; no longer U$1.PF0
- net DIO0: now also IC2.PB8; no longer U$1.PB8
- net DM: now also IC2.PA11, JP3.D+; no longer JP4.D+, U$1.PA11
- net DP: now also IC2.PA12, JP3.D-, R2.2; no longer JP4.D-, R4.2, U$1.PA12
- net GND: now also C2.2, C7.2, IC2.VSS, IC2.VSS2, IC2.VSSA, IC3.GND, JP3.VBUS, JP4.6, R1.1; no longer C11.2, C6.2, IC2.GND, JP3.6, JP4.VBUS, R2.1, U$1.VSS, U$1.VSS2, U$1.VSSA
- net GPIO0: now also IC2.PA0; no longer U$1.PA0
- net GPIO15: now also IC2.PA1; no longer U$1.PA1
- net I2C2_SCL: now also IC2.PB10, IC3.SCK, R5.1; no longer IC2.SCK, R1.1, U$1.PB10
- net I2C2_SDA: now also IC2.PB11, IC3.DATA, R4.1; no longer IC2.DATA, R5.1, U$1.PB11
- net MISO: now also IC2.PB4; no longer U$1.PB4
- net MOSI: now also IC2.PB5; no longer U$1.PB5
- net N$10: now also RN1B.2; no longer RN1C.2
- net N$11: now also C6.1, IC2.VDDIO; no longer C2.1, U$1.VDDIO
- net N$12: now also IC2.PA5; no longer U$1.PA5
- net N$13: now also C6.2, IC2.VSS1; no longer C2.2, U$1.VSS1
- net N$14: now also IC2.PA6; no longer U$1.PA6
- net N$15: now also IC2.BOOT0, R1.2; no longer R2.2, U$1.BOOT0
- net N$16: now also IC2.PA7; no longer U$1.PA7
- net N$17: now also IC2.PA10; no longer U$1.PA10
- net N$18: now also IC2.PA9, R2.1; no longer R4.1, U$1.PA9
- net N$2: now also IC2.PC13, RN1C.1; no longer RN1D.1, U$1.PC13
- net N$20: now also LED1.A, RN1C.2; no longer LED3.A, RN1D.2
- net N$21: now also IC2.PC14, RN1B.1; no longer RN1C.1, U$1.PC14
- net N$22: now also IC2.PC15, RN1A.1; no longer RN1B.1, U$1.PC15
- net N$26: now also IC2.PB13; no longer U$1.PB13
- net N$27: now also IC2.PB14; no longer U$1.PB14
- net N$8: now also IC2.PA4; no longer U$1.PA4
- net N$9: now also LED3.A; no longer LED1.A, RN1B.2
- net NRST: now also IC2.NRST; no longer U$1.NRST
- net NSS: now also IC2.PB9; no longer U$1.PB9
- net SCK: now also IC2.PB3; no longer U$1.PB3
- net SWCLK: now also IC2.PA14; no longer U$1.PA14
- net SWDAT: now also IC2.PA13; no longer U$1.PA13
- net USART1_RX: now also IC2.PB7; no longer U$1.PB7
- net USART1_TX: now also IC2.PB6; no longer U$1.PB6
- net USART2_RX: now also IC2.PA3, JP4.3; no longer JP3.3, U$1.PA3
- net USART2_TX: now also IC2.PA2, JP4.2; no longer JP3.2, U$1.PA2
- net VBUS: now also C1.1, JP3.GND; no longer C8.1, JP4.GND
- net W_RST: now also IC2.PF1; no longer U$1.PF1
Other:
- moved on the sheet: C1, C10, C2, C3, C4, C5, C6, C8, C9, LED1, LED3, R1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

Commit message: increasing cap package size
Parts:
- C5: device rcl:C-EUC0603 -> rcl:C-EUC0805
Changed lines of the file:
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@@
 <part name="+3V5" library="supply1" deviceset="+3V3" device=""/>
 <part name="C1" library="rcl" deviceset="C-EU" device="C0603" value="4u7"/>
-<part name="C5" library="rcl" deviceset="C-EU" device="C0603" value="4u7"/>
+<part name="C5" library="rcl" deviceset="C-EU" device="C0805" value="4u7"/>
 <part name="GND11" library="supply1" deviceset="GND" device=""/>
 <part name="GND12" library="supply1" deviceset="GND" device=""/>
@@
 <instance part="R2" gate="G$1" x="165.1" y="91.44"/>
 <instance part="GND9" gate="1" x="177.8" y="91.44" rot="R270"/>
-<instance part="+3V5" gate="G$1" x="241.3" y="104.14" rot="R270"/>
+<instance part="+3V5" gate="G$1" x="248.92" y="104.14" rot="R270"/>
 <instance part="C1" gate="G$1" x="213.36" y="101.6"/>
 <instance part="C5" gate="G$1" x="238.76" y="101.6"/>
@@
 <pinref part="+3V5" gate="G$1" pin="+3V3"/>
 <pinref part="C5" gate="G$1" pin="1"/>
-<junction x="238.76" y="104.14"/>
+<junction x="246.38" y="104.14"/>
 <pinref part="IC1" gate="A1" pin="VO"/>
 <wire x1="236.22" y1="104.14" x2="238.76" y2="104.14" width="0.1524" layer="91"/>
-</segment>
-<segment>
+<junction x="238.76" y="104.14"/>
+<wire x1="246.38" y1="104.14" x2="238.76" y2="104.14" width="0.1524" layer="91"/>
+</segment>
+<segment>

Commit message: adding some values and labels
Other:
- note added: "ADD INDUCTOR"
Changed lines of the file:
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@@
 <text x="154.94" y="106.68" size="1.778" layer="91">NC if 072 used</text>
 <text x="58.42" y="167.64" size="1.778" layer="91">spec</text>
+<text x="205.74" y="96.52" size="1.778" layer="91" rot="R90">ADD INDUCTOR</text>
 </plain>
 <instances>

Commit message: almost done
Parts:
- added R6: 1k, passives-7351:RESISTOR0603-N
- added U$3: ESP-07, Mine:ESP-07
- added X3: LTI-SASF54GT, con-coax:LTI-SASF54GT
- added X4: SMA-142-0711-821/826, con-coax:SMA-142-0711-821/826
- added X5: SMA-142-0711-871/876, con-coax:SMA-142-0711-871/876
- added X6: BU-SMA-V, con-coax:BU-SMA-V
- C1, C10, C2, C3, C4, C7, C8, C9: device rcl:C-EUC0603 -> passives-7351:CAPACITOR0603-N
- C5: device rcl:C-EUC0805 -> passives-7351:CAPACITOR0805-N
- C6: device rcl:C-EUC0603K -> passives-7351:CAPACITOR0603-N
- R1, R2, R3, R4, R5: device rcl:R-EU_R0603 -> passives-7351:RESISTOR0603-N
Connections:
- new net N$1: R6.P$2, U$3.GPIO2, X1.GPIO2
- new net N$3: U$3.GPIO14, X1.GPIO14
- new net N$4: U$3.GPIO13, X1.GPIO13
- new net N$7: U$3.GPIO12, X1.GPIO12
- net +3V3: now also R4.P$2, R5.P$2, R6.P$1, U$3.VCC; no longer R4.2, R5.2
- net CH_PD: now also U$3.CH_PD
- net DM: now also R3.P$2; no longer R3.2
- net DP: now also R2.P$2; no longer R2.2
- net GND: now also R1.P$1, U$3.GND; no longer R1.1
- net GPIO0: now also U$3.GPIO0
- net GPIO15: now also U$3.GPIO15
- net I2C2_SCL: now also R5.P$1; no longer R5.1
- net I2C2_SDA: now also R4.P$1; no longer R4.1
- net N$15: now also R1.P$2; no longer R1.2
- net N$17: now also R3.P$1; no longer R3.1
- net N$18: now also R2.P$1; no longer R2.1
- net USART1_RX: now also U$3.UTXD
- net USART1_TX: now also U$3.URXD
- net W_RST: now also U$3.GPIO16

Commit message: routed RST
Parts:
- removed SV1: (no value), con-lstb:MA04-2
- removed U$1: LMT85, Mine:LMT85
- removed X3: LTI-SASF54GT, con-coax:LTI-SASF54GT
- removed X4: SMA-142-0711-821/826, con-coax:SMA-142-0711-821/826
- removed X5: SMA-142-0711-871/876, con-coax:SMA-142-0711-871/876
- removed X6: BU-SMA-V, con-coax:BU-SMA-V
Connections:
- removed net N$5: SV1.5
- net +3V3: no longer SV1.2
- net CH_PD: no longer SV1.6
- net GND: no longer SV1.7
- net GPIO0: no longer SV1.3
- net RST: now also IC2.PA15
- net USART1_RX: no longer SV1.8
- net USART1_TX: no longer SV1.1
- net W_RST: no longer SV1.4
Changed lines of the file:
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@@
 <parts>
 <part name="IC2" library="dtb" deviceset="STM32F072" device=""/>
-<part name="SV1" library="con-lstb" deviceset="MA04-2" device=""/>
 <part name="U$2" library="hoperf" deviceset="RFM69HW" device=""/>
 <part name="JP1" library="SparkFun-Passives" deviceset="JUMPER-2" device="SMD-NC"/>
@@
 <part name="+3V8" library="supply1" deviceset="+3V3" device=""/>
 <part name="+3V9" library="supply1" deviceset="+3V3" device=""/>
-<part name="U$1" library="Mine" deviceset="LMT85" device=""/>
 <part name="IC3" library="Mine" deviceset="HTU21D" device=""/>
 <part name="+3V10" library="supply1" deviceset="+3V3" device=""/>
@@
 <part name="+3V15" library="supply1" deviceset="+3V3" device=""/>
 <part name="U$3" library="Mine" deviceset="ESP-07" device=""/>
-<part name="X3" library="con-coax" deviceset="LTI-SASF54GT" device=""/>
 <part name="GND23" library="supply1" deviceset="GND" device=""/>
 <part name="+3V16" library="supply1" deviceset="+3V3" device=""/>
-<part name="X4" library="con-coax" deviceset="SMA-" device="142-0711-821/826"/>
-<part name="X5" library="con-coax" deviceset="SMA-" device="142-0711-871/876"/>
-<part name="X6" library="con-coax" deviceset="BU-SMA-V" device=""/>
 </parts>
 <sheets>
@@
 <instances>
 <instance part="IC2" gate="G$1" x="93.98" y="68.58"/>
-<instance part="SV1" gate="G$1" x="99.06" y="165.1"/>
 <instance part="U$2" gate="A" x="172.72" y="180.34"/>
 <instance part="JP1" gate="A" x="53.34" y="78.74" rot="R90"/>
@@
 <instance part="+3V8" gate="G$1" x="180.34" y="119.38" rot="R90"/>
 <instance part="+3V9" gate="G$1" x="40.64" y="121.92"/>
-<instance part="U$1" gate="G$1" x="119.38" y="144.78"/>
 <instance part="IC3" gate="G$1" x="236.22" y="33.02"/>
 <instance part="+3V10" gate="G$1" x="241.3" y="50.8"/>
@@
 <instance part="+3V15" gate="G$1" x="68.58" y="210.82" rot="R90"/>
 <instance part="U$3" gate="G$1" x="30.48" y="210.82"/>
-<instance part="X3" gate="G$1" x="210.82" y="154.94" rot="MR0"/>
 <instance part="GND23" gate="1" x="30.48" y="185.42"/>
 <instance part="+3V16" gate="G$1" x="30.48" y="236.22"/>
-<instance part="X4" gate="G1" x="129.54" y="203.2"/>
-<instance part="X5" gate="G1" x="129.54" y="210.82"/>
-<instance part="X6" gate="G$1" x="127" y="220.98"/>
 </instances>
 <busses>
@@
 <net name="W_RST" class="0">
 <segment>
-<pinref part="SV1" gate="G$1" pin="4"/>
 <wire x1="91.44" y1="162.56" x2="71.12" y2="162.56" width="0.1524" layer="91"/>
 <label x="71.12" y="162.56" size="1.778" layer="95"/>
@@
 <net name="N$5" class="0">
 <segment>
-<pinref part="SV1" gate="G$1" pin="5"/>
 <wire x1="116.84" y1="165.1" x2="106.68" y2="165.1" width="0.1524" layer="91"/>
 </segment>
@@
 <net name="CH_PD" class="0">
 <segment>
-<pinref part="SV1" gate="G$1" pin="6"/>
 <wire x1="91.44" y1="165.1" x2="71.12" y2="165.1" width="0.1524" layer="91"/>
 <label x="71.12" y="165.1" size="1.778" layer="95"/>
@@
 </segment>
 <segment>
-<pinref part="SV1" gate="G$1" pin="7"/>
 <wire x1="106.68" y1="167.64" x2="116.84" y2="167.64" width="0.1524" layer="91"/>
 <pinref part="GND21" gate="1" pin="GND"/>
@@
 </segment>
 <segment>
-<pinref part="SV1" gate="G$1" pin="2"/>
 <wire x1="91.44" y1="160.02" x2="83.82" y2="160.02" width="0.1524" layer="91"/>
 <pinref part="C2" gate="G$1" pin="1"/>
@@
 <label x="139.7" y="185.42" size="1.778" layer="95"/>
 </segment>
+<segment>
+<pinref part="IC2" gate="G$1" pin="PA15"/>
+<wire x1="124.46" y1="91.44" x2="137.16" y2="91.44" width="0.1524" layer="91"/>
+<label x="129.54" y="91.44" size="1.778" layer="95"/>
+</segment>
 </net>
 <net name="N$2" class="0">
@@
 </segment>
 <segment>
-<pinref part="SV1" gate="G$1" pin="8"/>
 <wire x1="91.44" y1="167.64" x2="71.12" y2="167.64" width="0.1524" layer="91"/>
 <label x="71.12" y="167.64" size="1.778" layer="95"/>
@@
 </segment>
 <segment>
-<pinref part="SV1" gate="G$1" pin="1"/>
 <wire x1="106.68" y1="160.02" x2="129.54" y2="160.02" width="0.1524" layer="91"/>
 <label x="121.92" y="160.02" size="1.778" layer="95"/>
@@
 </segment>
 <segment>
-<pinref part="SV1" gate="G$1" pin="3"/>
 <wire x1="106.68" y1="162.56" x2="129.54" y2="162.56" width="0.1524" layer="91"/>
 <label x="121.92" y="162.56" size="1.778" layer="95"/>
