File: board/magnet-node.brd (EAGLE design)
At the start: 24 x 23 mm, 32 parts, among them IC1 MSP430G2X21, IC2 HTU21D, IC3 SI4012

Commit message: adding stencil and couple of values
Parts:
- C4: value (none) -> 100n
Changed lines of the file:
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@@
 </element>
 <element name="IC2" library="Mine" package="DFN6-L" value="HTU21D" x="22.22" y="12.5" smashed="yes"/>
-<element name="C4" library="passives-7351" package="C0603-N" value="" x="22.098" y="16.002" smashed="yes" rot="R180">
+<element name="C4" library="passives-7351" package="C0603-N" value="100n" x="22.098" y="16.002" smashed="yes" rot="R180">
 <attribute name="NAME" x="20.60890625" y="16.372921875" size="1.016" layer="25" font="vector" ratio="14" rot="R180"/>
 </element>

Commit message: fixing value
Parts:
- C10: value 47n -> 2n2
Changed lines of the file:
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@@
 <attribute name="NAME" x="20.60890625" y="18.404921875" size="1.016" layer="25" font="vector" ratio="14" rot="R180"/>
 </element>
-<element name="C10" library="passives-7351" package="C0603-N" value="47n" x="22.098" y="20.066" smashed="yes">
+<element name="C10" library="passives-7351" package="C0603-N" value="2n2" x="22.098" y="20.066" smashed="yes">
 <attribute name="NAME" x="20.79309375" y="20.965078125" size="1.016" layer="25" font="vector" ratio="14"/>
 </element>
