File: board-mrf89/mrf89-breakout.sch (EAGLE design)
At the start: 21 parts, among them IC1 MRF89XA

Commit message: pretty much done
Parts:
- added U$4: CRYSTAL-GROUNDED, SparkFun-FreqCtrl:CRYSTAL-GROUNDED
- added U$5: BOARD-RADIO, Mine:BOARD-RADIO
- C1: value (none) -> 220n
- C10: value (none) -> 100n
- C2, C4: value (none) -> 1u
- C3: value (none) -> 47n
- C5: value (none) -> 100p
- C8: value (none) -> 680p
- C9: value (none) -> 10n
- L1: value (none) -> 100n; device passives-7351:INDUCTOR0402-N -> passives-7351:INDUCTOR0603-N
- L2, L4: value (none) -> 6.8n
- R1: value (none) -> 1
- R2: value (none) -> 100k
- R3: value (none) -> 6.8k
Connections:
- removed net N$13: U$2.2, U$3.ANT
- removed net N$18: IC1.SCK, U$3.SCK
- removed net N$19: IC1.SDO, U$3.MISO
- removed net N$20: IC1.SDI, U$3.MOSI
- removed net N$21: IC1.CSDAT, U$3.NSS
- removed net N$22: IC1.CSCON, U$3.RESET
- removed net N$23: IC1.IRQ0, U$3.DIO0
- new net ANT: U$2.2, U$5.10
- new net CSDAT: IC1.CSDAT, U$5.1
- new net IRQ0: IC1.IRQ0, U$5.2
- new net MISO: IC1.SDO, U$5.13
- new net MOSI: IC1.SDI, U$5.14
- new net N$38: U$5.16
- new net NSS: IC1.CSCON, U$5.15
- new net SCK: IC1.SCK, U$5.12
- net +3V3: now also U$5.8; no longer U$3.VCC
- net DIO1: now also U$5.3; no longer U$3.DIO1
- net DIO2: now also U$5.4; no longer U$3.DIO2
- net DIO3: now also U$5.5; no longer U$3.DIO3
- net DIO4: now also U$5.6; no longer U$3.DIO4
- net DIO5: now also U$5.7; no longer U$3.DIO5
- net GND: now also U$4.3, U$5.11, U$5.9; no longer U$3.GNDA, U$3.GNDB
- net N$16: now also U$4.1
- net N$17: now also U$4.2
Other:
- note added: "2373927"
- moved on the sheet: C6
