File: board-35/tx35-pnl.brd (EAGLE design)
At the start: 38.1 x 15.6 mm, 32 parts, among them IC1 STM32F030K6, J1 SWD_SHROUD, Q1 MOSFET-NCHANNEL2N7002PW, X1 SMA-142-0711-821/826

Commit message: addin gvalues
Parts:
- L1: value 2u2 -> (none)
Other:
- board size 38.1 x 15.6 mm -> 46.9 x 24.4 mm
- board text added: "C1"
- board text added: "C10"
- board text added: "C11"
- board text added: "C12"
- board text added: "C13"
- board text added: "C2"
- board text added: "C3"
- board text added: "C4"
- board text added: "C5"
- board text added: "C6"
- board text added: "C7"
- board text added: "C8"
- board text added: "C9"
- board text added: "D1"
- board text added: "IC1"
- board text added: "JP2"
- board text added: "L1"
- board text added: "L2"
- board text added: "L3"
- board text added: "Q1"
- board text added: "R1"
- board text added: "R2"
- board text added: "R4"
- board text added: "X1"
- board text added: "Y1"
